File: PCB/stepper_driver/DRV8825_Driver/DRV8825_Driver.kicad_sch (KiCad schematic)
At the start: 21 parts, among them J1 Conn_01x04_Pin, J2 Conn_01x02_Pin, J3 Conn_01x02_Pin, SW1 SW_DIP_x03, U1 DRV8825PWP

Commit message: blah
Parts:
- removed C4, C5: 0.1u, Capacitor_SMD:C_0603_1608Metric, symbol Device:C
- removed J3: Conn_01x02_Pin, Connector_JST:JST_XH_B2B-XH-A_1x02_P2.50mm_Vertical, symbol Connector:Conn_01x02_Pin
- added J3: Conn_01x03_Pin, Connector_JST:JST_XH_B3B-XH-A_1x03_P2.50mm_Vertical, symbol Connector:Conn_01x03_Pin
- added J5: USB_C_Receptacle_PowerOnly_6P, Connector_USB:USB_C_Receptacle_GCT_USB4135-GF-A_6P_TopMnt_Horizontal, symbol Connector:USB_C_Receptacle_PowerOnly_6P
- C1: footprint Capacitor_SMD:C_0603_1608Metric -> Capacitor_SMD:C_0805_2012Metric
- C3: footprint Capacitor_SMD:C_0603_1608Metric -> Capacitor_SMD:C_0805_2012Metric_Pad1.18x1.45mm_HandSolder
- C7: value 0.47uF -> 0.47uF 6.3v; footprint Capacitor_SMD:C_0603_1608Metric -> Capacitor_SMD:C_0805_2012Metric_Pad1.18x1.45mm_HandSolder
- J2: footprint TerminalBlock_4Ucon:TerminalBlock_4Ucon_1x02_P3.50mm_Horizontal -> TerminalBlock_Phoenix:TerminalBlock_Phoenix_MKDS-1,5-2_1x02_P5.00mm_Horizontal
- R10, R11, R5, R6, R9: footprint Resistor_SMD:R_0603_1608Metric -> Resistor_SMD:R_0805_2012Metric
- R4: footprint Resistor_SMD:R_0603_1608Metric -> Capacitor_SMD:C_0805_2012Metric
Connections:
- net 3V3: no longer SW1.4, SW1.5, SW1.6
- net DIR: now also J3.1 (Pin_1)
- net STEP: now also J3.2 (Pin_2)
- net gnd!: now also J3.3 (Pin_3), J5.A12 (GND), J5.B12 (GND), J5.S1 (SHIELD)
- new net VUSB: J5.A9 (VBUS), J5.B9 (VBUS), SW1.4, SW1.5, SW1.6
Other:
- moved on the sheet: C3
