File: PCB/stepper_driver/DRV8825_Driver/_autosave-DRV8825_Driver.kicad_pcb (KiCad board)
At the start: 2 copper layers, 36 x 33.3 mm, 24 parts, among them J1 Conn_01x04_Pin, J2 Conn_01x02_Pin, J3 Conn_01x03_Pin, J5 USB_C_Receptacle_PowerOnly_6P, SW1 SW_DIP_x03, U1 DRV8825PWP

Commit message: blah
Parts:
- C1, R4: footprint Capacitor_SMD:C_0805_2012Metric -> Capacitor_SMD:C_0805_2012Metric_Pad1.18x1.45mm_HandSolder
- C2, C4, C5: footprint Capacitor_SMD:C_0603_1608Metric -> Capacitor_SMD:C_0805_2012Metric_Pad1.18x1.45mm_HandSolder
- R7, R8: footprint Resistor_SMD:R_0603_1608Metric -> Resistor_SMD:R_0805_2012Metric
- moved why??? 12.3 mm to (48.0, 79.6)
- moved R5 1.10 mm to (52.1, 79.1)
- moved R6 0.92 mm to (52.0, 76.0)
- moved C7 0.84 mm to (37.6, 87.3)
- moved R4 0.60 mm to (39.3, 80.8)
- moved C3 0.45 mm to (39.3, 76.8)
- moved C2 0.36 mm to (41.8, 80.7)
- moved C5 0.36 mm to (43.5, 76.9)
- moved R7 0.27 mm to (38.0, 89.3)
- moved C4 0.24 mm to (41.4, 76.8)
- moved R8 0.22 mm to (38.0, 91.3)
- moved R11 0.20 mm to (54.0, 87.0)
- moved C1 0.20 mm to (52.7, 83.0)
Routing:
- net gnd!: track 57.2 -> 62.1 mm, vias 16 -> 14
- net M0: track 23.9 -> 26.3 mm
- net VCP: track 22.1 -> 20.1 mm
- net M1: track 17.5 -> 19.3 mm
- net VMA: track 45.2 -> 43.6 mm, vias 2 -> 4
- net M2: track 11.5 -> 13.1 mm
- net ISENA: track 6.43 -> 7.45 mm
- net ISENB: track 10.8 -> 11.7 mm
Other:
- board text removed: "J2"
