File: PCB/stepper_driver/DRV8825_Driver/_autosave-DRV8825_Driver.kicad_sch (KiCad schematic)
At the start: 21 parts, among them J1 Conn_01x04_Pin, J2 Conn_01x02_Pin, J3 Conn_01x03_Pin, SW1 SW_DIP_x03, U1 DRV8825PWP

Commit message: blah
Parts:
- removed C4, C5: 0.1u, Capacitor_SMD:C_0603_1608Metric, symbol Device:C
- added J5: USB_C_Receptacle_PowerOnly_6P, Connector_USB:USB_C_Receptacle_GCT_USB4135-GF-A_6P_TopMnt_Horizontal, symbol Connector:USB_C_Receptacle_PowerOnly_6P
- C1: footprint Capacitor_SMD:C_0603_1608Metric -> Capacitor_SMD:C_0805_2012Metric
- C3: footprint Capacitor_SMD:C_0603_1608Metric -> Capacitor_SMD:C_0805_2012Metric_Pad1.18x1.45mm_HandSolder
- C7: value 0.47uF -> 0.47uF 6.3v; footprint Capacitor_SMD:C_0603_1608Metric -> Capacitor_SMD:C_0805_2012Metric_Pad1.18x1.45mm_HandSolder
- J2: footprint TerminalBlock_4Ucon:TerminalBlock_4Ucon_1x02_P3.50mm_Horizontal -> TerminalBlock_Phoenix:TerminalBlock_Phoenix_MKDS-1,5-2_1x02_P5.00mm_Horizontal
- R10, R11, R5, R6, R8, R9: footprint Resistor_SMD:R_0603_1608Metric -> Resistor_SMD:R_0805_2012Metric
- R4, R7: footprint Resistor_SMD:R_0603_1608Metric -> Capacitor_SMD:C_0805_2012Metric
Connections:
- net 3V3: no longer SW1.4, SW1.5, SW1.6
- net gnd!: now also J5.A12 (GND), J5.B12 (GND), J5.S1 (SHIELD)
- new net VUSB: J5.A9 (VBUS), J5.B9 (VBUS), SW1.4, SW1.5, SW1.6
Other:
- moved on the sheet: C3
Changed lines of the file:
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@@
 	)
 	(junction
-		(at 27.94 130.81)
-		(diameter 0)
-		(color 0 0 0 0)
-	)
-	(junction
 		(at 27.94 109.22)
 		(diameter 0)
@@
 	)
 	(junction
-		(at 27.94 138.43)
+		(at 27.94 106.68)
 		(diameter 0)
 		(color 0 0 0 0)
 	)
 	(junction
-		(at 27.94 106.68)
+		(at 107.95 49.53)
 		(diameter 0)
 		(color 0 0 0 0)
@@
 	(wire
 		(pts
-			(xy 27.94 138.43) (xy 36.83 138.43)
-		)
-		(stroke
-			(width 0)
-			(type default)
-		)
-	)
-	(wire
-		(pts
 			(xy 30.48 158.75) (xy 33.02 158.75)
 		)
@@
 	(wire
 		(pts
-			(xy 19.05 130.81) (xy 27.94 130.81)
-		)
-		(stroke
-			(width 0)
-			(type default)
-		)
-	)
-	(wire
-		(pts
 			(xy 99.06 137.16) (xy 106.68 137.16)
 		)
@@
 	(wire
 		(pts
-			(xy 19.05 138.43) (xy 27.94 138.43)
+			(xy 34.29 109.22) (xy 27.94 109.22)
 		)
 		(stroke
@@
 	(wire
 		(pts
-			(xy 34.29 109.22) (xy 27.94 109.22)
+			(xy 55.88 104.14) (xy 55.88 106.68)
 		)
 		(stroke
@@
 	(wire
 		(pts
-			(xy 55.88 104.14) (xy 55.88 106.68)
+			(xy 104.14 49.53) (xy 107.95 49.53)
 		)
 		(stroke
@@
 	(wire
 		(pts
+			(xy 107.95 49.53) (xy 107.95 50.8)
+		)
+		(stroke
+			(width 0)
+			(type default)
+		)
+	)
+	(wire
+		(pts
 			(xy 99.06 137.16) (xy 99.06 142.24)
 		)
@@
 	(wire
 		(pts
-			(xy 27.94 130.81) (xy 36.83 130.81)
+			(xy 127 24.13) (xy 129.54 24.13)
 		)
 		(stroke
@@
 	(wire
 		(pts
+			(xy 107.95 49.53) (xy 111.76 49.53)
+		)
+		(stroke
+			(width 0)
+			(type default)
+		)
+	)
+	(wire
+		(pts
 			(xy 90.17 104.14) (xy 95.25 104.14)
 		)
@@
 		)
 	)
+	(global_label "VUSB"
+		(shape input)
+		(at 129.54 24.13 270)
+		(fields_autoplaced yes)
+		(effects
+			(font
+				(size 1.27 1.27)
+			)
+			(justify right)
+		)
+		(property "Intersheetrefs" "${INTERSHEET_REFS}"
+			(at 129.54 32.0138 90)
+			(effects
+				(font
+					(size 1.27 1.27)
+				)
+				(justify right)
+				(hide yes)
+			)
+		)
+	)
 	(global_label "BVREF"
 		(shape input)
@@
 		)
 	)
-	(global_label "3V3"
+	(global_label "VUSB"
 		(shape input)
 		(at 59.69 137.16 180)
@@
 		)
 		(property "Intersheetrefs" "${INTERSHEET_REFS}"
-			(at 53.1972 137.16 0)
+			(at 51.8062 137.16 0)
 			(effects
 				(font
@@
 		)
 	)
+	(global_label "gnd!"
+		(shape input)
+		(at 107.95 50.8 270)
+		(fields_autoplaced yes)
+		(effects
+			(font
+				(size 1.27 1.27)
+			)
+			(justify right)
+		)
+		(property "Intersheetrefs" "${INTERSHEET_REFS}"
+			(at 107.95 57.837 90)
+			(effects
+				(font
+					(size 1.27 1.27)
+				)
+				(justify right)
+				(hide yes)
+			)
+		)
+	)
 	(global_label "M2"
 		(shape input)
@@
 	(symbol
 		(lib_id "Device:C")
-		(at 19.05 134.62 0)
+		(at 27.94 134.62 0)
 		(unit 1)
 		(exclude_from_sim no)
@@
 		(dnp no)
 		(property "Reference" "C3"
-			(at 21.336 134.874 0)
+			(at 30.226 134.874 0)
 			(effects
 				(font
@@
 		)
 		(property "Value" "4.7u"
-			(at 21.336 136.652 0)
+			(at 30.226 136.652 0)
 			(effects
 				(font
@@
 			)
 		)
-		(property "Footprint" "Capacitor_SMD:C_0603_1608Metric"
-			(at 20.0152 138.43 0)
+		(property "Footprint" "Capacitor_SMD:C_0805_2012Metric_Pad1.18x1.45mm_HandSolder"
+			(at 28.9052 138.43 0)
 			(effects
 				(font
@@
 		)
 		(property "Datasheet" "~"
-			(at 19.05 134.62 0)
+			(at 27.94 134.62 0)
 			(effects
 				(font
@@
 		)
 		(property "Description" "Unpolarized capacitor"
-			(at 19.05 134.62 0)
+			(at 27.94 134.62 0)
 			(effects
 				(font
@@
 			)
 		)
-		(property "Footprint" "Resistor_SMD:R_0603_1608Metric"
+		(property "Footprint" "Resistor_SMD:R_0805_2012Metric"
 			(at 91.44 65.532 90)
 			(effects
@@
 			)
 		)
-		(property "Footprint" "TerminalBlock_4Ucon:TerminalBlock_4Ucon_1x02_P3.50mm_Horizontal"
+		(property "Footprint" "TerminalBlock_Phoenix:TerminalBlock_Phoenix_MKDS-1,5-2_1x02_P5.00mm_Horizontal"
 			(at 38.1 167.64 0)
 			(effects
@@
 			)
 		)
-		(property "Footprint" "Resistor_SMD:R_0603_1608Metric"
+		(property "Footprint" "Capacitor_SMD:C_0805_2012Metric"
 			(at 54.102 100.33 90)
 			(effects
@@
 	)
 	(symbol
-		(lib_id "Device:C")
-		(at 27.94 134.62 0)
-		(unit 1)
-		(exclude_from_sim no)
-		(in_bom yes)
-		(on_board yes)
-		(dnp no)
-		(property "Reference" "C4"
-			(at 29.972 134.874 0)
-			(effects
-				(font
-					(size 1.27 1.27)
-				)
-				(justify left)
-			)
-		)
-		(property "Value" "0.1u"
-			(at 30.226 136.652 0)
-			(effects
-				(font
-					(size 1.27 1.27)
-				)
-				(justify left)
-			)
-		)
-		(property "Footprint" "Capacitor_SMD:C_0603_1608Metric"
-			(at 28.9052 138.43 0)
-			(effects
-				(font
-					(size 1.27 1.27)
-				)
-				(hide yes)
-			)
-		)
-		(property "Datasheet" "~"
-			(at 27.94 134.62 0)
-			(effects
-				(font
-					(size 1.27 1.27)
-				)
-				(hide yes)
-			)
-		)
-		(property "Description" "Unpolarized capacitor"
-			(at 27.94 134.62 0)
-			(effects
-				(font
-					(size 1.27 1.27)
-				)
-				(hide yes)
-			)
-		)
-		(pin "2"
-		)
-		(pin "1"
-		)
-		(instances
-			(project "DRV8825_Driver"
-				(path "/ee279c60-8c91-429e-ac7b-9a9136d33130"
-					(reference "C4")
-					(unit 1)
-				)
-			)
-		)
-	)
-	(symbol
 		(lib_id "Connector:Conn_01x04_Pin")
 		(at 38.1 156.21 0)
@@
 			)
 		)
-		(property "Footprint" "Resistor_SMD:R_0603_1608Metric"
+		(property "Footprint" "Resistor_SMD:R_0805_2012Metric"
 			(at 95.25 133.858 90)
 			(effects
@@
 			)
 		)
-		(property "Footprint" "Resistor_SMD:R_0603_1608Metric"
+		(property "Footprint" "Resistor_SMD:R_0805_2012Metric"
 			(at 91.44 70.612 90)
 			(effects
@@
 		(dnp no)
 		(property "Reference" "C7"
-			(at 77.47 62.738 0)
+			(at 77.978 62.484 0)
 			(effects
 				(font
@@
 			)
 		)
-		(property "Value" "0.47uF"
-			(at 77.47 65.278 0)
+		(property "Value" "0.47uF 6.3v"
+			(at 77.978 60.452 0)
 			(effects
 				(font
@@
 			)
 		)
-		(property "Footprint" "Capacitor_SMD:C_0603_1608Metric"
+		(property "Footprint" "Capacitor_SMD:C_0805_2012Metric_Pad1.18x1.45mm_HandSolder"
 			(at 86.0552 66.04 0)
 			(effects
@@
 			)
 		)
-		(property "Footprint" "Resistor_SMD:R_0603_1608Metric"
+		(property "Footprint" "Resistor_SMD:R_0805_2012Metric"
 			(at 54.102 113.03 90)
 			(effects
@@
 			)
 		)
-		(property "Footprint" "Capacitor_SMD:C_0603_1608Metric"
+		(property "Footprint" "Capacitor_SMD:C_0805_2012Metric"
 			(at 86.0552 29.21 0)
 			(effects
@@
 			)
 		)
-		(property "Footprint" "Resistor_SMD:R_0603_1608Metric"
+		(property "Footprint" "Capacitor_SMD:C_0805_2012Metric"
 			(at 32.512 113.03 90)
 			(effects
@@
 			)
 		)
-		(property "Footprint" "Resistor_SMD:R_0603_1608Metric"
+		(property "Footprint" "Resistor_SMD:R_0805_2012Metric"
 			(at 95.25 144.018 90)
 			(effects
@@
 	)
 	(symbol
-		(lib_id "Device:C")
-		(at 36.83 134.62 0)
+		(lib_id "Connector:USB_C_Receptacle_PowerOnly_6P")
+		(at 111.76 31.75 0)
 		(unit 1)
 		(exclude_from_sim no)
@@
 		(on_board yes)
 		(dnp no)
-		(property "Reference" "C5"
-			(at 39.37 134.3661 0)
+		(fields_autoplaced yes)
+		(property "Reference" "J5"
+			(at 111.76 13.97 0)
 			(effects
 				(font
 					(size 1.27 1.27)
 				)
-				(justify left)
 			)
 		)
-		(property "Value" "0.1u"
-			(at 39.624 136.398 0)
+		(property "Value" "USB_C_Receptacle_PowerOnly_6P"
+			(at 111.76 16.51 0)
 			(effects
 				(font
 					(size 1.27 1.27)
 				)
-				(justify left)
 			)
 		)
-		(property "Footprint" "Capacitor_SMD:C_0603_1608Metric"
-			(at 37.7952 138.43 0)
+		(property "Footprint" "Connector_USB:USB_C_Receptacle_GCT_USB4135-GF-A_6P_TopMnt_Horizontal"
+			(at 115.57 29.21 0)
 			(effects
 				(font
@@
 			)
 		)
-		(property "Datasheet" "~"
-			(at 36.83 134.62 0)
+		(property "Datasheet" "https://www.usb.org/sites/default/files/documents/usb_type-c.zip"
+			(at 111.76 31.75 0)
 			(effects
 				(font
@@
 			)
 		)
-		(property "Description" "Unpolarized capacitor"
-			(at 36.83 134.62 0)
+		(property "Description" "USB Power-Only 6P Type-C Receptacle connector"
+			(at 111.76 31.75 0)
 			(effects
 				(font
@@
 			)
 		)
-		(pin "2"
+		(pin "A9"
 		)
-		(pin "1"
+		(pin "B12"
+		)
+		(pin "A12"
+		)
+		(pin "B5"
+		)
+		(pin "B9"
+		)
+		(pin "S1"
+		)
+		(pin "A5"
 		)
 		(instances
-			(project "DRV8825_Driver"
+			(project ""
 				(path "/ee279c60-8c91-429e-ac7b-9a9136d33130"
-					(reference "C5")
+					(reference "J5")
 					(unit 1)
 				)
@@
 			)
 		)
-		(property "Footprint" "Resistor_SMD:R_0603_1608Metric"
+		(property "Footprint" "Resistor_SMD:R_0805_2012Metric"
 			(at 95.25 138.938 90)
 			(effects
